Commit message: feat(sim): export link meshes and regenerated URDF
STL units verified as mm via tools/check_stl.py (wheel bbox 101.0);
mesh scale 0.001 confirmed. Fusion doc saved as JetAcker_Sim.

File: EdgeAIJetson/Sim_Resources/urdf/jetacker.urdf (robot description, URDF)
Before this commit: robot jetacker, 13 links, 12 joints
Links:
- link base_link: mass 4 -> 4.05
